File: wireless_timer/pcb/combined.brd (EAGLE design)
At the start: 36 x 76.5 mm, 51 parts, among them U1 ATTINY1616-SNR

Commit message: dcdc added
Parts:
- removed D1: BAT, diode:SOD-123_MINI-SMA
- removed R20: 30K, rcl:R0805
- removed R21: 200E, rcl:R0805
- added C12: 10uF, rcl:C0805
- moved C8 6.90 mm to (10.7, 44.5), turned to 270 degrees
- moved R19 0.14 mm to (25.7, 24.0)
Connections:
- removed net N$3: JP3.1, R21.2
- removed net SHDN: R20.2, U1.6
- removed net VADC: C1.1, R1.1, R2.1, U1.2
- new net M0: U1.19
- new net VA: U1.7
- new net VB: C1.1, R1.1, R2.1, U1.4
- new net VC: U1.5
- net GND: now also C12.2; no longer R20.1
- net RXD1: now also U1.17; no longer U1.18
- net S4: now also U1.3; no longer U1.19
- net S6: now also U1.6; no longer U1.4
- net SET: now also U1.2; no longer U1.7
- net TXD1: now also U1.18; no longer U1.17
- net VBAT: no longer D1.A
- net VCC: now also JP3.1, JP5.1, R6.2, TP2.TP, U1.1; no longer A1.1, C10.1, C11.1, JP1.3, R17.1, R18.1
- net VDD: now also A1.1, C10.1, C11.1, C12.1, JP1.3, R17.1, R18.1; no longer D1.C, JP5.1, R21.1, R6.2, TP2.TP, U1.1
