File: wireless_timer/pcb/combined.sch (EAGLE design)
At the start: 122 parts, among them Q1 MMBT2222A, U1 ATTINY1616-SNR, U2 DMP3165L, U3 DMP3165L, U4 ATTINY1616-SNR, U5 AMS1117-3.3, U6 DMP3165L, U7 DMP3165L, U8 DMP3165L, U9 DMP3165L

Commit message: layout cleaned
Parts:
- removed C12, C21, C22, C23, C24: 100nF, rcl:C-EUC0603K
- removed C13, C14, C15, C16, C17, C18, C19, C20, C25, C26, C27: 10uF, rcl:C-EUC0805
- removed CHG, TPVAO: TPTP18R, testpad:TPTP18R
- removed D2, D3: CGRM4005-G, diode:CGRM4005-G
- removed H1, H10, H2, H3, H4, H6, H8, H9: MOUNT-HOLE3.2, holes:MOUNT-HOLE3.2
- removed HC0, HC1, HC12: 1X05, pinhead_smd:1X05
- removed OLED, PCU, PCUT: (no value), pinhead-2:PINHD-1X04_2.54-S
- removed Q1: MMBT2222A, MMBT2222A:MMBT2222A
- removed R22, R23, R24, R25, R26, R27, R29, R30, R31, R32, R33, R34, R35, R36, R37: 10K, rcl:R-US_R0603
- removed R28: 10k, rcl:R-US_R0603
- removed R38, R39, R40, R41: 499E, rcl:R-US_R0603
- removed S10, S7, S8, S9: SW_55MM, switch_5p5mm:SW_55MM
- removed TMR: (no value), pinhead-2:PINHD-1X08_2.54-S
- removed U2, U3, U6, U7, U8, U9: DMP3165L, DMP3165L:DMP3165L
- removed U4: ATTINY1616-SNR, ATTINY1616-SNR:ATTINY1616-SNR
- removed U5: AMS1117-3.3, AMS1117-3.3:AMS1117-3.3
- removed UPD, UPDT: (no value), pinhead-2:PINHD-1X03_2.54-S
- removed VIN, VOUT: (no value), pinhead:PINHD-1X2
- removed VOUT2: (no value), pinhead-2:PINHD-1X02_2.54-S
- added A1: 1X05, pinhead_smd:1X05
- added JP5: (no value), pinhead-2:PINHD-1X04_2.54-S
- C1, C7: device rcl:C-EUC0603K -> rcl:C-EUC0805
- C10, C11, C8: value 100nF -> 10uF; device rcl:C-EUC0603K -> rcl:C-EUC0805
- C2, C3, C4, C5: value 10uF -> 100nF
- C6: value 10uF -> 100nF; device rcl:CPOL-USCT3528 -> rcl:C-EUC0805
- C9: value 100nF -> 10uF; device rcl:C-EUC0603K -> rcl:CPOL-USCT3528
- D1: value CGRM4005-G -> BAT
- JP1: device pinhead-2:PINHD-1X06_2.54-S -> pinhead-2:PINHD-1X04_2.54-S
- JP2: device pinhead:PINHD-1X5 -> pinhead-2:PINHD-1X02_2.54-S
- JP3: device pinhead-2:PINHD-1X06_2.54-S -> pinhead-2:PINHD-1X03_2.54-S
- R1, R2: value 1K -> 100K; device rcl:R-US_R0603 -> rcl:R-US_R0805
- R10: value 1K -> 10K; device rcl:R-US_R0603 -> rcl:R-US_R0805
- R11, R7, R8, R9: value 30K -> 10K; device rcl:R-US_R0603 -> rcl:R-US_R0805
- R12, R13, R14: device rcl:R-US_R0603 -> rcl:R-US_R0805
- R15, R16: value 10K -> 1K; device rcl:R-US_R0603 -> rcl:R-US_R0805
- R17, R18, R19, R20: value 10K -> 30K; device rcl:R-US_R0603 -> rcl:R-US_R0805
- R21: value 10K -> 200E; device rcl:R-US_R0603 -> rcl:R-US_R0805
- R3, R4: value 100K -> 10K; device rcl:R-US_R0603 -> rcl:R-US_R0805
- R5, R6: value 1K -> 10K
- renumbered 5V to TP2, BAT+ to TP4, BAT- to TP5, GND to TP1, K to TP3, VOUT1 to JP4
Connections:
- removed net +12V: TMR.1, U7.D, U9.D, VOUT.1
- removed net 12VIN: C25.1, C27.1, R25.2, U5.VIN, U7.S, U9.S, VIN.1
- removed net 12V_EN: R26.1, U4.PB1/SDA
- removed net AX: TMR.2, U4.PA4/SS
- removed net BX: TMR.3, U4.PA5
- removed net CX: TMR.4, U4.PA6
- removed net DX: TMR.5, U4.PA7
- removed net EX: TMR.6, U4.PB5
- removed net FX: TMR.7, U4.PB4
- removed net M0: U1.PA3/SCK, U2.G
- removed net M0_T: U4.PA3/SCK, U6.G
- removed net M1_T: R39.2, U4.PC0, U8.G
- removed net M1_T0: C23.1, R35.1, R39.1
- removed net M1_T1: JP1.2, JP2.2, JP3.2, R34.1, R35.2, S9.1, S9.2
- removed net N$11: Q1.B, R26.2, R27.1
- removed net N$13: Q1.C, R28.2
- removed net N$14: D3.C, U8.S
- removed net N$17: R25.1, R28.1, U7.G, U9.G
- removed net N$23: U4.PA0/RESET/UPDI, UPDT.2
- removed net N$4: R10.2, R11.1, U3.G
- removed net N$6: D2.C, U6.S
- removed net RXD0PC: PCUT.3, U4.PB3/RXD0
- removed net RXD0_T: HC0.4, U4.PA2/MISO/RXD1
- removed net RXD1_T: HC1.4, R40.2, U4.PC1
- removed net RXD1_T0: C22.1, R33.1, R40.1
- removed net RXD1_T1: JP1.3, JP2.3, JP3.3, R32.1, R33.2, S8.1, S8.2
- removed net SET0_T: HC0.5, R24.2, U4.PC3
- removed net SET1_T: HC1.5, R29.2, R38.2, U4.PB0/SCL
- removed net SET1_T0: C24.1, R37.1, R38.1
- removed net SET1_T1: JP1.1, JP2.1, JP3.1, R36.1, R37.2, S10.1, S10.2
- removed net TXD0PC: PCUT.2, U4.PB2/TXD0
- removed net TXD0_T: HC0.3, U4.PA1/MOSI/TXD1
- removed net TXD1_T: HC1.3, R41.2, U4.PC2
- removed net TXD1_T0: C21.1, R31.1, R41.1
- removed net TXD1_T1: JP1.4, JP2.4, JP3.4, R30.1, R31.2, S7.1, S7.2
- removed net UPDI: U1.PA0/RESET/UPDI, UPD.2
- removed net VA: R2.1, U1.PB4
- removed net VAO: R2.2, TPVAO.TP
- removed net VB: C1.1, R3.1, R4.1, U1.PA6
- removed net VC: R1.1, U1.PA7
- removed net VCHG: CHG.TP, R1.2
- removed net VDD0: C13.1, C14.1, C15.1, HC0.1, U6.D
- removed net VDD1: C17.1, C18.1, C19.1, HC1.1, U8.D
- new net SHDN: R20.2, U1.PB5
- new net VADC: C1.1, R1.1, R2.1, U1.PA4/SS
- net GND: now also A1.2, C6.2, C9.-, JP1.4, JP2.2, JP3.2, JP5.4, R19.1, R2.2, R20.1; no longer C12.2, C13.2, C14.2, C15.2, C16.2, C17.2, C18.2, C19.2, C20.2, C21.2, C22.2, C23.2, C24.2, C25.2, C26.2, C27.2, C6.-, C9.2, HC0.2, HC1.2, HC12.2, JP1.5, JP2.5, JP3.5, JP3.6, OLED.4, PCU.4, PCUT.4, Q1.E, R11.2, R24.1, R27.2, R29.1, R4.2, R7.1, S10.3, S10.4, S7.3, S7.4, S8.3, S8.4, S9.3, S9.4, TMR.8, U4.GND, U5.GND/ADJ, UPD.3, UPDT.3, VIN.2, VOUT.2, VOUT2.2
- net N$1: now also R5.2, R6.1, S1.1, S1.2; no longer R13.1, R15.2, S6.1, S6.2
- net N$10: now also R10.1, R8.2; no longer R18.1, R21.2
- net N$12: now also R3.1, R4.2, S2.1, S2.2; no longer R12.1, R14.2, S1.1, S1.2
- net N$2: now also JP3.3, U1.PA0/RESET/UPDI; no longer D1.C, U2.S
- net N$3: now also JP3.1, R21.2; no longer OLED.3, U3.D
- net N$5: now also R11.2, R12.1, S4.1, S4.2; no longer R17.1, R20.2, S2.1, S2.2
- net N$8: now also R13.2, R14.1, S6.1, S6.2; no longer R22.1, R23.2, S3.1, S3.2
- net N$9: now also R7.1, R9.2, S3.1, S3.2; no longer R16.1, R19.2, S4.1, S4.2
- net RXD0: now also R15.2; no longer R10.1, R6.2
- net RXD00: now also JP5.3, R15.1; no longer PCU.3, R6.1
- net RXD1: now also A1.4, U1.PA2/MISO/RXD1; no longer HC12.4, U1.PA1/MOSI/TXD1
- net S1: now also C2.1, R4.1; no longer C7.1, R14.1
- net S2: now also C6.1, R11.1; no longer C10.1, R20.1
- net S3: now also C7.1, R13.1; no longer C12.1, R23.1
- net S4: now also C5.1, R9.1, U1.PA3/SCK; no longer C9.1, R19.1, U1.PA5
- net S5: now also C4.1, R8.1; no longer C11.1, R21.1
- net S6: now also C3.1, R5.1, U1.PA6; no longer C8.1, R15.1, U1.PB5
- net SCL: now also JP1.2, R18.2; no longer JP1.6, OLED.2, R8.2
- net SDA: now also JP1.1, R17.2; no longer OLED.1, R9.2
- net SET: now also A1.5, R19.2, U1.PB4; no longer HC12.5, R7.2, U1.PA4/SS
- net TXD0: now also R16.2; no longer R5.2
- net TXD00: now also JP5.2, R16.1; no longer PCU.2, R5.1
- net TXD1: now also A1.3, U1.PA1/MOSI/TXD1; no longer HC12.3, U1.PA2/MISO/RXD1
- net VBAT: now also D1.A, JP2.1, R1.2; no longer R3.2, VOUT2.1
- net VCC: now also A1.1, C10.1, C11.1, C8.1, C9.+, JP1.3, R10.2, R14.2, R17.1, R18.1, R3.2, R7.2; no longer C16.1, C20.1, C26.1, C5.1, C6.+, D1.A, D2.A, D3.A, PCU.1, PCUT.1, R13.2, R16.2, R17.2, R18.2, R22.2, R30.2, R32.2, R34.2, R36.2, R8.1, R9.1, TP2.TP, U1.VDD, U3.S, U4.VDD, U5.VOUT, UPD.1, UPDT.1
- net VDD: now also D1.C, JP5.1, R21.1, R6.2, TP2.TP, U1.VDD; no longer C2.1, C3.1, C4.1, HC12.1, U2.D

Commit message: dcdc added
Parts:
- removed C8: 10uF, rcl:C-EUC0805
- removed R20: 30K, rcl:R-US_R0805
- added C17, C18, C19: 10uF, rcl:C-EUC0805
- added D2: SS22, SS22:SS22
- added L1: 1u, 5040_INDUCTOR:5040_INDUCTOR
- added R38: 511K, rcl:R-US_M0805
- added R39: 91K, rcl:R-US_M0805
- added R42, R45: 50K, rcl:R-US_M0805
- added U2: TPS, TPS63000DRLR:TPS563212DRLR
Connections:
- new net LX1: L1.2, U2.LX1
- new net LX2: L1.1, U2.LX2
- new net N$27: R38.1, R39.2, U2.FB
- new net N$37: R42.2, U2.MODE
- new net VINPUT: C17.1, D2.K, U2.VIN
- net GND: now also C17.2, C18.2, C19.2, R39.1, R42.1, R45.1, U2.GND; no longer C8.2, R20.1
- net SHDN: now also R45.2, U2.EN; no longer R20.2
- net VCC: now also C18.1, C19.1, R38.2, U2.VOUT; no longer C8.1
- net VDD: now also D2.A
