File: wireless_timer/pcb/combined.sch (EAGLE design)
At the start: 50 parts, among them U1 ATTINY1616-SNR

Commit message: layout completed
Parts:
- added C17, C18, C19: 10uF, rcl:C-EUC0805
- added D2, D3: BAT, diode:CGRM4005-G
- added JP6, JP7: (no value), pinhead-2:PINHD-1X02_2.54-S
- added L1: 1uH, 5040_INDUCTOR:5040_INDUCTOR
- added R22, R23: 100K, rcl:R-US_R0805
- added R38: 511K, rcl:R-US_M0805
- added R39: 91K, rcl:R-US_M0805
- added R45: 50K, rcl:R-US_M0805
- added U2: TPS, TPS63000DRLR:TPS563212DRLR
- added U3, U4: PMOS, DMP3165L:DMP3165L
- S1, S2, S3, S4, S5, S6: value SW_55MM -> SW
- TP1, TP5: value TPTP18R -> GND
- TP2: value TPTP18R -> VDD
- TP3: value TPTP18R -> VCC
- TP4: value TPTP18R -> VBAT
- U1: value ATTINY1616-SNR -> 1
Connections:
- new net DC_SW: R22.1, U1.PA5, U3.G
- new net LX1: L1.2, U2.LX1
- new net LX2: L1.1, U2.LX2
- new net N$27: R38.1, R39.2, U2.FB
- new net N$36: R45.2, U2.EN
- new net VBAT_O: D1.A, D3.A, JP6.2, JP7.2, R1.2, R22.2, U3.S
- new net VCC_SW: R23.2, U1.PA7, U4.G
- new net VIN: C17.1, D3.C, U2.VIN, U3.D
- net GND: now also C17.2, C18.2, C19.2, R39.1, R45.1, U2.GND
- net S6: no longer TP3.TP
- net SHDN: now also U2.MODE
- net VBAT: now also JP6.1, JP7.1; no longer D1.A, R1.2
- net VCC: now also C18.1, C19.1, D2.A, R23.1, R38.2, TP3.TP, U2.VOUT, U4.S
- net VDD: now also D2.C, U4.D
