File: wireless_timer/pcb/dcdc.brd (EAGLE design)
At the start: 8 parts, among them U2 TPS

Commit message: layout completed
Other:
- board text removed: "BAT"
- board text removed: "Dadabhagwan.org"
- board text removed: "G"
- board text removed: "I2C"
- board text removed: "LI_UART1"
- board text removed: "PC_UART0"
- board text removed: "UPD0"
- board text removed: "UPD1"
